Commit message: Added scorpius base

File: urdf/scorpius.xacro (robot description, xacro)
@@ -2,8 +2,11 @@
     xmlns:xacro="http://www.ros.org/wiki/xacro">
     <xacro:macro name="scorpius" params="base_link">
+        <xacro:include filename="$(find scorpius_base_description)/urdf/scorpius_base_description.xacro" />
         <xacro:include filename="$(find sting_description)/urdf/sting.xacro" />
         <xacro:include filename="$(find sting_carriage_description)/urdf/sting_carriage.xacro" />
+        <xacro:property name="carriage_base" value="carriage_link_base" />
         <xacro:property name="payload" value="payload" />
-        <xacro:sting_carriage base_link="${base_link}" payload="${payload}" />
+        <xacro:scorpius_base_description base_link="${base_link}" carriage_base="${carriage_base}" />
+        <xacro:sting_carriage base_link="${carriage_base}" payload="${payload}" />
         <xacro:sting base_link="${payload}" />
     </xacro:macro>
